File: MMCProMicro.kicad_pcb (KiCad board)
At the start: 2 copper layers, 17.8 x 33 mm, 20 parts, among them J1 USB2_C_Receptacle, J2 Conn_01x12, J3 Conn_01x12, U1 ATmega32U4-AU, X1 Crystal_GND2

Commit message: Rev.B
Parts:
- added TP3: TestPoint, proj_local:Measurement_Point_RoundSquare-TH_Tiny, F.Cu at (29.8, 48.2)
- D1: footprint proj_local:D_0603_HandSoldering -> proj_local:D_TUMD2_HandSoldering
- X1: value Crystal_GND2 -> Resonator; footprint proj_local:Resonator_SMD_muRata_CSTxExxV-3Pin_3.0x1.1mm_HandSoldering -> proj_local:Resonator_SMD_muRata_CSTxExxV-3Pin_3.0x1.1mm_HandSoldering_Compact
- moved D1 0.87 mm to (19.9, 27.4)
- moved R1 0.47 mm to (21.5, 30.3)
- moved R2 0.31 mm to (22.9, 30.3)
- moved R5 0.13 mm to (19.8, 32.6)
- moved R3 0.09 mm to (24.2, 30.0)
- moved R4 0.09 mm to (25.6, 30.0)
- moved C5 0.08 mm to (20.7, 47.0)
- moved C6 0.08 mm to (30.1, 47.0)
- moved X1 0.08 mm to (25.4, 47.7)
- moved TP1 0.07 mm to (23.8, 32.5)
Routing:
- net GND: track 21.0 -> 20.1 mm, vias 19 -> 18
- net VCC: track 50.7 -> 49.9 mm
Other:
- board text added: "Rev.B"
- board text removed: "Rev.A"

Commit message: Rev.C
Connections:
- U1 pad 33: Net-(U1-Pad33) -> GND
Routing:
- net GND: track 20.1 -> 21.3 mm
Other:
- net class GND: trace_width 0.25 -> 0.2
- board text added: "Rev.C"
- board text removed: "Rev.B"

Commit message: Rev.D
Parts:
- added G***: LOGO, proj_local:ShiroMicroLogo, B.Cu at (25.2, 33.7)
- added JP1: SolderJumper_2_Open, proj_local:SolderJumper-2_P1.0mm_Open_RoundedPad0.7x1.0mm, F.Cu at (30.4, 25.3)
- added JP2: SolderJumper_2_Open, proj_local:SolderJumper-2_P1.0mm_Open_RoundedPad0.7x1.0mm, F.Cu at (22.1, 48.6)
- added TP4: TestPoint, proj_local:Measurement_Point_RoundSquare-TH_Tiny, F.Cu at (31.2, 34.6)
- C1, C4, C5, C6: footprint Capacitors_SMD:C_0603_HandSoldering -> proj_local:C_0603_HandSoldering
- C2: renamed from C3; footprint Capacitors_SMD:C_0603_HandSoldering -> proj_local:C_0603_HandSoldering
- C3: renamed from C2; footprint Capacitors_SMD:C_0603_HandSoldering -> proj_local:C_0603_HandSoldering
- F1: footprint Resistors_SMD:R_0805_HandSoldering -> proj_local:F_0805_HandSoldering
- R1, R2, R3, R4, R5: footprint Resistors_SMD:R_0603_HandSoldering -> proj_local:R_0603_HandSoldering
- U1: footprint Package_QFP:TQFP-44_10x10mm_P0.8mm -> proj_local:TQFP-44_10x10mm_P0.8mm
- moved R4 0.42 mm to (26.0, 30.0)
- moved F1 0.34 mm to (25.2, 26.8)
- moved TP1 0.25 mm to (23.9, 32.3)
- moved R3 0.23 mm to (24.5, 30.0)
- moved C2 0.20 mm to (27.8, 29.8)
- moved C3 0.10 mm to (29.4, 29.8)
- moved R1 0.10 mm to (21.4, 30.3)
- moved R2 0.08 mm to (22.9, 30.3)
Connections:
- J3 pad 1: VBUS -> /NC
- U1 pad 26: Net-(U1-Pad26) -> /PD6
Routing:
- net PD7: track 14.6 -> 9.97 mm
- net PE6: track 24.8 -> 20.3 mm
- net /PD6: track 0.00 -> 4.53 mm
- net PB4: track 12.9 -> 9.73 mm
- net VBUS: track 31.1 -> 28.4 mm
- net XTAL1: track 11.3 -> 13.5 mm
- net /NC: track 0.00 -> 2.06 mm
- net XTAL2: track 15.7 -> 14.4 mm
- net Net-(J1-PadA5): track 8.35 -> 7.20 mm
- net Net-(J1-PadA7): track 7.71 -> 6.74 mm
- net GND: track 21.3 -> 22.0 mm, vias 18 -> 17
- net PB5: track 17.4 -> 18.1 mm
- added copper zone on F.Cu, net /NC
- removed copper zone on F.Cu, net VBUS
Other:
- board text added: "NC"
- board text added: "PD6"
- board text added: "Rev.D"
- board text removed: "RAW"
- board text removed: "Rev.C"
